Commit message: Remove unnecessary floating point from joint axes
Signed-off-by: Andrej Orsula <orsula.andrej@gmail.com>

File: urdf/ur5_rg2.urdf (robot description, URDF)
Before this commit: robot ur5_rg2, 11 links, 10 joints
Joints:
- joint shoulder_pan_joint: axis 0.0 0.0 1.0 -> 0 0 1
- joint wrist_2_joint: axis 0.0 0.0 1.0 -> 0 0 1
